Commit message: Fixed rover design, should be pretty much accurate

File: description/robot_core.xacro (robot description, xacro)
@@ -7,5 +7,5 @@
     <material name="orange">
         <color rgba=" 1 0.3 0.1 1"/>
-    </material>
+    </material>For
     <material name="blue">
         <color rgba=" 0.2 0.2 1 1"/>
@@ -22,5 +22,5 @@
         <parent link="base_link"/>
         <child link="chassis"/>
-        <origin xyz="-0.089 0 0"/>
+        <origin xyz="0 0 0"/>
     </joint>
     <link name="chassis">
@@ -48,5 +48,5 @@
         <parent link="base_link"/>
         <child link="left_front_wheel"/>
-        <origin xyz=" 0 .0635 0" rpy="-${pi/2} 0 0"/>
+        <origin xyz="0.122 .02 -0.125" rpy="-${pi/2} 0 0"/>
         <axis xyz="0 0 1"/>
     </joint>
@@ -55,5 +55,5 @@
             <origin xyz="0 0 0.0381"/>
             <geometry>
-                <cylinder radius="0.025" length="0.04"/>
+                <cylinder radius="0.05" length="0.08"/>
             </geometry>
             <material name="blue"/>
@@ -62,8 +62,8 @@
             <origin xyz="0 0 0.0381"/>
             <geometry>
-                <cylinder radius="0.025" length="0.04"/>
-            </geometry>
-        </collision>
-        <xacro:inertial_cylinder mass="0.1" length="0.04" radius=".025">
+                <cylinder radius="0.05" length="0.08"/>
+            </geometry>
+        </collision>
+        <xacro:inertial_cylinder mass="0.1" length="0.08" radius=".05">
             <origin xyz="0 0 0.0" rpy="0 0 0"/>
         </xacro:inertial_cylinder>
@@ -75,5 +75,5 @@
         <parent link="base_link"/>
         <child link="right_front_wheel"/>
-        <origin xyz=" 0 -0.127 0" rpy="-${pi/2} 0 0"/>
+        <origin xyz="0.122 -.02 -0.125" rpy="${pi/2} 0 0"/>
         <axis xyz="0 0 -1"/>
     </joint>
@@ -82,5 +82,5 @@
             <origin xyz="0 0 0.0381"/>
             <geometry>
-                <cylinder radius="0.025" length="0.04"/>
+                <cylinder radius="0.05" length="0.08"/>
             </geometry>
             <material name="blue"/>
@@ -89,8 +89,8 @@
             <origin xyz="0 0 0.0381"/>
             <geometry>
-                <cylinder radius="0.025" length="0.04"/>
-            </geometry>
-        </collision>
-        <xacro:inertial_cylinder mass="0.1" length="0.04" radius=".025">
+                <cylinder radius="0.05" length="0.08"/>
+            </geometry>
+        </collision>
+        <xacro:inertial_cylinder mass="0.1" length="0.08" radius=".05">
             <origin xyz="0 0 0.0" rpy="0 0 0"/>
         </xacro:inertial_cylinder>
@@ -99,15 +99,15 @@
         <material>Gazebo/Blue</material>
     </gazebo>
-    <joint name="left_back_wheel_joint" type="continuous">
-        <parent link="base_link"/>
-        <child link="left_back_wheel"/>
-        <origin xyz="-0.128 .0635 0" rpy="-${pi/2} 0 0"/>
+    <joint name="left_middle_wheel_joint" type="continuous">
+        <parent link="base_link"/>
+        <child link="left_middle_wheel"/>
+        <origin xyz="0 .02 -0.125" rpy="-${pi/2} 0 0"/>
         <axis xyz="0 0 1"/>
     </joint>
-    <link name="left_back_wheel">
-        <visual>
-            <origin xyz="0 0 0.0381"/>
-            <geometry>
-                <cylinder radius="0.025" length="0.04"/>
+    <link name="left_middle_wheel">
+        <visual>
+            <origin xyz="0 0 0.0381"/>
+            <geometry>
+                <cylinder radius="0.05" length="0.08"/>
             </geometry>
             <material name="blue"/>
@@ -116,11 +116,65 @@
             <origin xyz="0 0 0.0381"/>
             <geometry>
-                <cylinder radius="0.025" length="0.04"/>
-            </geometry>
-        </collision>
-        <xacro:inertial_cylinder mass="0.1" length="0.04" radius=".025">
+                <cylinder radius="0.05" length="0.08"/>
+            </geometry>
+        </collision>
+        <xacro:inertial_cylinder mass="0.1" length="0.08" radius="0.05">
             <origin xyz="0 0 0.0" rpy="0 0 0"/>
         </xacro:inertial_cylinder>
     </link>
+    <gazebo reference="left_middle_wheel">
+        <material>Gazebo/Blue</material>
+    </gazebo>
+    <joint name="right_middle_wheel_joint" type="continuous">
+        <parent link="base_link"/>
+        <child link="right_middle_wheel"/>
+        <origin xyz="0 -.02 -0.125" rpy="${pi/2} 0 0"/>
+        <axis xyz="0 0 -1"/>
+    </joint>
+    <link name="right_middle_wheel">
+        <visual>
+            <origin xyz="0 0 0.0381"/>
+            <geometry>
+                <cylinder radius="0.05" length="0.08"/>
+            </geometry>
+            <material name="blue"/>
+        </visual>
+        <collision>
+            <origin xyz="0 0 0.0381"/>
+            <geometry>
+                <cylinder radius="0.05" length="0.08"/>
+            </geometry>
+        </collision>
+        <xacro:inertial_cylinder mass="0.1" length="0.08" radius=".05">
+            <origin xyz="0 0 0.0" rpy="0 0 0"/>
+        </xacro:inertial_cylinder>
+    </link>
+    <gazebo reference="right_middle_wheel">
+        <material>Gazebo/Blue</material>
+    </gazebo>
+    <joint name="left_back_wheel_joint" type="continuous">
+        <parent link="base_link"/>
+        <child link="left_back_wheel"/>
+        <origin xyz="-0.118 .03 -0.125" rpy="-${pi/2} 0 0"/>
+        <axis xyz="0 0 1"/>
+    </joint>
+    <link name="left_back_wheel">
+        <visual>
+            <origin xyz="0 0 0.0381"/>
+            <geometry>
+                <cylinder radius="0.05" length="0.08"/>
+            </geometry>
+            <material name="blue"/>
+        </visual>
+        <collision>
+            <origin xyz="0 0 0.0381"/>
+            <geometry>
+                <cylinder radius="0.05" length="0.08"/>
+            </geometry>
+        </collision>
+        <xacro:inertial_cylinder mass="0.1" length="0.08" radius=".05">
+            <origin xyz="0 0 0" rpy="0 0 0"/>
+        </xacro:inertial_cylinder>
+    </link>
     <gazebo reference="left_back_wheel">
         <material>Gazebo/Blue</material>
@@ -129,5 +183,5 @@
         <parent link="base_link"/>
         <child link="right_back_wheel"/>
-        <origin xyz=" -0.128 -0.127 0" rpy="-${pi/2} 0 0"/>
+        <origin xyz=" -0.118 -.03 -0.125" rpy="${pi/2} 0 0"/>
         <axis xyz="0 0 -1"/>
     </joint>
@@ -136,5 +190,5 @@
             <origin xyz="0 0 0.0381"/>
             <geometry>
-                <cylinder radius="0.025" length="0.04"/>
+                <cylinder radius="0.05" length="0.08"/>
             </geometry>
             <material name="blue"/>
@@ -143,8 +197,8 @@
             <origin xyz="0 0 0.0381"/>
             <geometry>
-                <cylinder radius="0.025" length="0.04"/>
-            </geometry>
-        </collision>
-        <xacro:inertial_cylinder mass="0.1" length="0.04" radius=".025">
+                <cylinder radius="0.05" length="0.08"/>
+            </geometry>
+        </collision>
+        <xacro:inertial_cylinder mass="0.1" length="0.08" radius=".05">
             <origin xyz="0 0 0.0" rpy="0 0 0"/>
         </xacro:inertial_cylinder>
@@ -154,2 +208,367 @@
     </gazebo>
 </robot>
+<!-- This URDF was automatically created by SolidWorks to URDF Exporter! Originally created by Stephen Brawner (brawner@gmail.com)
+     Commit Version: 1.6.0-4-g7f85cfe  Build Version: 1.6.7995.38578
+     For more information, please see http://wiki.ros.org/sw_urdf_exporter -->
+<!-- <robot xmlns:xacro="http://www.ros.org/wiki/xacro">
+    <xacro:include filename="inertial_macros.xacro"/>
+    name="my_bot">
+  <link
+    name="base_link">
+    <inertial>
+      <origin
+        xyz="0.18096 0.13921 0.16741"
+        rpy="0 0 0" />
+      <mass
+        value="0.39929" />
+      <inertia
+        ixx="0.0011054"
+        ixy="9.6361E-07"
+        ixz="1.8822E-16"
+        iyy="0.0023993"
+        iyz="1.9082E-15"
+        izz="0.0017729" />
+    </inertial>
+    <visual>
+      <origin
+        xyz="0 0 0"
+        rpy="0 0 0" />
+      <geometry>
+        <mesh
+          filename="package://ARGGG/meshes/base_link.STL" />
+      </geometry>
+      <material
+        name="">
+        <color
+          rgba="0.89804 0.91373 0.92549 1" />
+      </material>
+    </visual>
+    <collision>
+      <origin
+        xyz="0 0 0"
+        rpy="0 0 0" />
+      <geometry>
+        <mesh
+          filename="package://ARGGG/meshes/base_link.STL" />
+      </geometry>
+    </collision>
+  </link>
+  <link
+    name="Empty_Link1">
+    <inertial>
+      <origin
+        xyz="0.028575 8.5594E-06 -0.0635"
+        rpy="0 0 0" />
+      <mass
+        value="0.019306" />
+      <inertia
+        ixx="1.2326E-06"
+        ixy="3.2731E-15"
+        ixz="3.2296E-22"
+        iyy="1.2326E-06"
+        iyz="-1.6399E-22"
+        izz="1.9461E-06" />
+    </inertial>
+    <visual>
+      <origin
+        xyz="0 0 0"
+        rpy="0 0 0" />
+      <geometry>
+        <mesh
+          filename="package://ARGGG/meshes/Empty_Link1.STL" />
+      </geometry>
+      <material
+        name="">
+        <color
+          rgba="0.79216 0.81961 0.92941 1" />
+      </material>
+    </visual>
+    <collision>
+      <origin
+        xyz="0 0 0"
+        rpy="0 0 0" />
+      <geometry>
+        <mesh
+          filename="package://ARGGG/meshes/Empty_Link1.STL" />
+      </geometry>
+    </collision>
+  </link>
+  <joint
+    name="1"
+    type="continuous">
+    <origin
+      xyz="0.18119 -0.23091 0.14969"
+      rpy="1.5708 0.00029954 0" />
+    <parent
+      link="base_link" />
+    <child
+      link="Empty_Link1" />
+    <axis
+      xyz="0 0 0" />
+  </joint>
+  <link
+    name="Empty_Link2">
+    <inertial>
+      <origin
+        xyz="0.12139 0.026219 -0.0762"
+        rpy="0 0 0" />
+      <mass
+        value="0.22286" />
+      <inertia
+        ixx="0.00030845"
+        ixy="0.0002357"
+        ixz="1.2212E-12"
+        iyy="0.0010487"
+        iyz="-8.3429E-12"
+        izz="0.0013512" />
+    </inertial>
+    <visual>
+      <origin
+        xyz="0 0 0"
+        rpy="0 0 0" />
+      <geometry>
+        <mesh
+          filename="package://ARGGG/meshes/Empty_Link2.STL" />
+      </geometry>
+      <material
+        name="">
+        <color
+          rgba="0.49804 0.49804 0.49804 1" />
+      </material>
+    </visual>
+    <collision>
+      <origin
+        xyz="0 0 0"
+        rpy="0 0 0" />
+      <geometry>
+        <mesh
+          filename="package://ARGGG/meshes/Empty_Link2.STL" />
+      </geometry>
+    </collision>
+  </link>
+  <joint
+    name="2"
+    type="continuous">
+    <origin
+      xyz="-0.044434 -0.053353 0.0127"
+      rpy="0 0 0.00029954" />
+    <parent
+      link="Empty_Link1" />
+    <child
+      link="Empty_Link2" />
+    <axis
+      xyz="0 0 0" />
+  </joint>
+  <link
+    name="Empty_Link3">
+    <inertial>
+      <origin
+        xyz="0 1.3567E-06 0.003175"
+        rpy="0 0 0" />
+      <mass
+        value="0.0042119" />
+      <inertia
+        ixx="3.2106E-07"
+        ixy="5.1796E-13"
+        ixz="5.3789E-12"
+        iyy="3.2146E-07"
+        iyz="-6.6644E-18"
+        izz="6.1434E-07" />
+    </inertial>
+    <visual>
+      <origin
+        xyz="0 0 0"
+        rpy="0 0 0" />
+      <geometry>
+        <mesh
+          filename="package://ARGGG/meshes/Empty_Link3.STL" />
+      </geometry>
+      <material
+        name="">
+        <color
+          rgba="0.64706 0.61961 0.58431 1" />
+      </material>
+    </visual>
+    <collision>
+      <origin
+        xyz="0 0 0"
+        rpy="0 0 0" />
+      <geometry>
+        <mesh
+          filename="package://ARGGG/meshes/Empty_Link3.STL" />
+      </geometry>
+    </collision>
+  </link>
+  <joint
+    name="3"
+    type="continuous">
+    <origin
+      xyz="0.01905 0.01524 0.0127"
+      rpy="0 0 0.39034" />
+    <parent
+      link="Empty_Link2" />
+    <child
+      link="Empty_Link3" />
+    <axis
+      xyz="0 0 0" />
+  </joint>
+  <link
+    name="Empty_Link4">
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
File: description/ros2_control.xacro (robot description, xacro)
@@ -14,4 +14,20 @@
         </joint>
         <joint name="right_front_wheel_joint">
+            <command_interface name="velocity">
+                <param name="min">-10</param>
+                <param name="max">10</param>
+            </command_interface>
+            <state_interface name="velocity"/>
+            <state_interface name="position"/>
+        </joint>
+                <joint name="left_middle_wheel_joint">
+            <command_interface name="velocity">
+                <param name="min">-10</param>
+                <param name="max">10</param>
+            </command_interface>
+            <state_interface name="velocity"/>
+            <state_interface name="position"/>
+        </joint>
+        <joint name="right_middle_wheel_joint">
             <command_interface name="velocity">
                 <param name="min">-10</param>

Commit message: added initial slam tracking

File: description/robot_core.xacro (robot description, xacro)
@@ -19,4 +19,11 @@
     <link name="base_link">
     </link>
+    <joint name="base_footprint_joint" type = "fixed">
+      <parent link="base_link"/>
+      <child link="base_footprint"/>
+      <origin xyz="0 0 0" rpy="0 0 0"/>
+    </joint>
+    <link name="base_footprint">
+    </link>
     <joint name="chassis_joint" type="fixed">
         <parent link="base_link"/>

Commit message: working on get

File: description/robot_core.xacro (robot description, xacro)
@@ -106,11 +106,11 @@
         <material>Gazebo/Blue</material>
     </gazebo>
-    <joint name="left_middle_wheel_joint" type="continuous">
-        <parent link="base_link"/>
-        <child link="left_middle_wheel"/>
+    <joint name="left_middle_joint" type="continuous">
+        <parent link="base_link"/>
+        <child link="left_wheel"/>
         <origin xyz="0 .02 -0.125" rpy="-${pi/2} 0 0"/>
         <axis xyz="0 0 1"/>
     </joint>
-    <link name="left_middle_wheel">
+    <link name="left_heel">
         <visual>
             <origin xyz="0 0 0.0381"/>
@@ -130,14 +130,14 @@
         </xacro:inertial_cylinder>
     </link>
-    <gazebo reference="left_middle_wheel">
+    <gazebo reference="left_wheel">
         <material>Gazebo/Blue</material>
     </gazebo>
-    <joint name="right_middle_wheel_joint" type="continuous">
-        <parent link="base_link"/>
-        <child link="right_middle_wheel"/>
+    <joint name="right_wheel_joint" type="continuous">
+        <parent link="base_link"/>
+        <child link="right_wheel"/>
         <origin xyz="0 -.02 -0.125" rpy="${pi/2} 0 0"/>
         <axis xyz="0 0 -1"/>
     </joint>
-    <link name="right_middle_wheel">
+    <link name="right_wheel">
         <visual>
             <origin xyz="0 0 0.0381"/>
@@ -157,5 +157,5 @@
         </xacro:inertial_cylinder>
     </link>
-    <gazebo reference="right_middle_wheel">
+    <gazebo reference="right_wheel">
         <material>Gazebo/Blue</material>
     </gazebo>

Commit message: yadaya ya

File: description/robot_core.xacro (robot description, xacro)
@@ -112,5 +112,5 @@
         <axis xyz="0 0 1"/>
     </joint>
-    <link name="left_heel">
+    <link name="left_wheel">
         <visual>
             <origin xyz="0 0 0.0381"/>

Commit message: fixes

File: description/robot_core.xacro (robot description, xacro)
@@ -52,5 +52,5 @@
         <material>Gazebo/White</material>
     </gazebo>
-    <joint name="left_front_wheel_joint" type="continuous">
+    <!-- <joint name="left_front_wheel_joint" type="continuous">
         <parent link="base_link"/>
         <child link="left_front_wheel"/>
@@ -105,6 +105,6 @@
     <gazebo reference="right_front_wheel">
         <material>Gazebo/Blue</material>
-    </gazebo>
-    <joint name="left_middle_joint" type="continuous">
+    </gazebo> -->
+    <joint name="left_wheel_joint" type="continuous">
         <parent link="base_link"/>
         <child link="left_wheel"/>
@@ -160,5 +160,5 @@
         <material>Gazebo/Blue</material>
     </gazebo>
-    <joint name="left_back_wheel_joint" type="continuous">
+    <!-- <joint name="left_back_wheel_joint" type="continuous">
         <parent link="base_link"/>
         <child link="left_back_wheel"/>
@@ -213,5 +213,5 @@
     <gazebo reference="right_back_wheel">
         <material>Gazebo/Blue</material>
-    </gazebo>
+    </gazebo> -->
 </robot>
 <!-- This URDF was automatically created by SolidWorks to URDF Exporter! Originally created by Stephen Brawner (brawner@gmail.com)
